File: prj/Peripherals.kicad_sch (KiCad schematic)
At the start: 12 parts, among them J1 Conn_01x16_Pin, J2 Conn_01x16_Pin, SW1 TSA063G60-250

Commit message: PCB routed trial 2
Parts:
- added D4: LED GREEN, LED_SMD:LED_0603_1608Metric, symbol Device:LED
- added R6: 1k, Resistor_SMD:R_0603_1608Metric, symbol Device:R
- D1: value LED -> LED RED; LCSC (none) -> C2286
- D2: value LED -> LED BLUE; LCSC (none) -> C2288
- D3: value LED -> LED YELLOW; LCSC (none) -> C2290
- D5: renamed from D4; value LED -> LED RED; LCSC (none) -> C2286
- J1, J2: now left out of the parts list
- R1: value 470 -> 10k; footprint Resistor_SMD:R_0402_1005Metric -> Resistor_SMD:R_0603_1608Metric; LCSC (none) -> C25804
- R2, R3, R4: footprint Resistor_SMD:R_0402_1005Metric -> Resistor_SMD:R_0603_1608Metric; LCSC (none) -> C21190
- R5: value 1k -> 10k; footprint Resistor_SMD:R_0402_1005Metric -> Resistor_SMD:R_0603_1608Metric; LCSC (none) -> C25804
- SW1: LCSC (none) -> C294566
Connections:
- net +3V3: now also D5.2 (A)
- net GND: now also R6.2
- net LED_4: now also D4.2 (A); no longer D5.2 (A)
- new net: D4.1 (K), R6.1
Other:
- moved on the sheet: D5, R5
