File: prj/MCU.kicad_sch (KiCad schematic)
At the start: 22 parts, among them J4 TagConnect, SW2 TSA063G60-250, U2 nRF52832-QFxx, Y1 32.768kHz, Y2 32MHz

Commit message: PCB routed trial 2
Parts:
- removed AE1: Antenna, RF_Antenna:Texas_SWRA117D_2.4GHz_Left, symbol Device:Antenna
- removed Y2: 32MHz, Crystal:Crystal_SMD_2012-2Pin_2.0x1.2mm, symbol Device:Crystal
- added AE1: Antenna_Shield, RF_Antenna:Texas_SWRA117D_2.4GHz_Left, symbol Device:Antenna_Shield
- added Y2: XL7EL89CKI-111YLC-32M, Crystal:Crystal_SMD_2016-4Pin_2.0x1.6mm, symbol Device:Crystal_GND24
- C10: footprint Capacitor_SMD:C_0402_1005Metric -> Capacitor_SMD:C_0603_1608Metric
- C11, C5, C6: footprint Capacitor_SMD:C_0402_1005Metric -> Capacitor_SMD:C_0603_1608Metric; LCSC (none) -> C14663
- C12: LCSC (none) -> C40459
- C13: value 12p -> 18p; footprint Capacitor_SMD:C_0402_1005Metric -> Capacitor_SMD:C_0603_1608Metric; LCSC (none) -> C1647
- C14: value 12p -> 18p; footprint Capacitor_SMD:C_0402_1005Metric -> Capacitor_SMD:C_0603_1608Metric
- C15, C16: value 12p -> 10p; footprint Capacitor_SMD:C_0402_1005Metric -> Capacitor_SMD:C_0603_1608Metric; LCSC (none) -> C1634
- C7: LCSC (none) -> C1705
- C8: LCSC (none) -> C1592
- C9: footprint Capacitor_SMD:C_0402_1005Metric -> Capacitor_SMD:C_0603_1608Metric; LCSC (none) -> C14858
- L2: footprint Inductor_SMD:L_0402_1005Metric -> Inductor_SMD:L_0603_1608Metric; LCSC (none) -> C304267
- L3: footprint Inductor_SMD:L_0603_1608Metric -> Inductor_SMD:L_0805_2012Metric; LCSC (none) -> C18221303
- L4: LCSC (none) -> C14033
- R12: renamed from R11; footprint Resistor_SMD:R_0402_1005Metric -> Resistor_SMD:R_0603_1608Metric; LCSC (none) -> C25804
- SW2: LCSC (none) -> C294566
- U2: LCSC (none) -> C77540
- Y1: value 32.768kHz -> Q13FC13500004; LCSC (none) -> C32346
Connections:
- net GND: now also AE1.2 (Shield), Y2.2, Y2.4
- net XC1: now also Y2.1
- net XC2: now also Y2.3
- net RF: now reaches L4.2
- net RF: now also AE1.1 (A)

Commit message: v1 ready
Parts:
- C14: LCSC (none) -> C1647
Changed lines of the file:
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@@
 			)
 		)
-		(property "LCSC" ""
+		(property "LCSC" "C1647"
 			(at 217.17 99.06 0)
 			(effects
